Commit message: Update

File: RoboRTS_Gazebo/robots/infantry.gazebo.xacro (robot description, xacro)
@@ -36,4 +36,5 @@
     <material>Gazebo/Black</material>
     <turnGravityOff>false</turnGravityOff>
+    <!--<kinematic>1</kinematic>-->
   </gazebo>
   <gazebo reference="uwb_tag_link">
@@ -47,5 +48,5 @@
   <!-- hokuyo -->
   <gazebo reference="base_laser_link">
-    <sensor type="gpu_ray" name="head_hokuyo_sensor">
+    <sensor type="ray" name="head_hokuyo_sensor">
       <pose>0 0 0.2 0 0 0</pose>
       <visualize>false</visualize>
@@ -54,6 +55,6 @@
         <scan>
           <horizontal>
-            <samples>360</samples>
-            <resolution>1</resolution>
+            <samples>720</samples>
+            <resolution>0.5</resolution>
             <min_angle>-3.14159</min_angle>
             <max_angle>3.14159</max_angle>
@@ -72,8 +73,8 @@
                reading. -->
           <mean>0.0</mean>
-          <stddev>0.01</stddev>
+          <stddev>0.015</stddev>
         </noise>
       </ray>
-      <plugin name="gazebo_ros_head_hokuyo_controller" filename="libgazebo_ros_gpu_laser.so">
+      <plugin name="gazebo_ros_head_hokuyo_controller" filename="libgazebo_ros_laser.so">
         <topicName>scan</topicName>
         <frameName>base_laser_link</frameName>
@@ -83,20 +84,34 @@
   <!-- position controller plugin-->
   <gazebo>
-    <plugin name="mecanum_base_controller" filename="libgazebo_ros_planar_move.so">
-      <commandTopic>cmd_vel</commandTopic>
-      <odometryTopic>odom</odometryTopic>
-      <odometryFrame>odom</odometryFrame>
-      <odometryRate>15</odometryRate>
-      <robotBaseFrame>base_link</robotBaseFrame>
-      <broadcastTF>true</broadcastTF>
+    <plugin name="mecanum_base_controller" filename="libroborts_gazebo_ros_force_based_omni_move.so">
+      <cmd_vel_topic>/cmd_vel</cmd_vel_topic>
+      <odom_topic>odom</odom_topic>
+      <odom_frame>odom</odom_frame>
+      <odom_rate>20.0</odom_rate>
+      <robot_base_frame>base_link</robot_base_frame>
+      <publish_odom_tf>1</publish_odom_tf>
+      <rotation_velocity_p_gain>800.0</rotation_velocity_p_gain>
    </plugin>
  </gazebo>
+  <!--<gazebo>-->
+  <!--<plugin name="mecanum_base_controller" filename="libroborts_gazebo_ros_force_based_move.so">-->
+  <!--<commandTopic>/cmd_vel</commandTopic>-->
+  <!--<odometryTopic>odom</odometryTopic>-->
+  <!--<odometryFrame>odom</odometryFrame>-->
+  <!--<odometryRate>20.0</odometryRate>-->
+  <!--<robotBaseFrame>base_link</robotBaseFrame>-->
+  <!--<yaw_velocity_p_gain>500</yaw_velocity_p_gain>-->
+  <!--<x_velocity_p_gain>3000</x_velocity_p_gain>-->
+  <!--<y_velocity_p_gain>3000</y_velocity_p_gain>-->
+  <!--<publishOdometryTf>1</publishOdometryTf>-->
+  <!--</plugin>-->
+  <!--</gazebo>-->
   <gazebo>
     <plugin name="uwb_plugin" filename="libroborts_gazebo_ros_uwb.so">
       <topic_name>uwb</topic_name>
       <frame_id>uwb</frame_id>
-      <body_name>uwb_tag_link</body_name>
-      <gaussian_noise>0.09</gaussian_noise>
-      <!--<update_rate_hz>50.0</update_rate_hz>-->
+      <body_name>base_link</body_name>
+      <gaussian_noise>0.04</gaussian_noise>
+      <update_rate_hz>15.0</update_rate_hz>
     </plugin>
   </gazebo>
@@ -121,9 +136,9 @@
   </gazebo>
 <!-- ros_control plugin -->
-  <gazebo>
-    <plugin name="gazebo_ros_control" filename="libgazebo_ros_control.so">
-      <robotParam>robot_description</robotParam>
+  <!--<gazebo>-->
+    <!--<plugin name="gazebo_ros_control" filename="libgazebo_ros_control.so">-->
+      <!--<robotParam>robot_description</robotParam>-->
      <!-- <robotSimType>gazebo_ros_control/DefaultRobotHWSim</robotSimType>-->
-    </plugin>
-  </gazebo>
+    <!--</plugin>-->
+  <!--</gazebo>-->
 </robot>

File: RoboRTS_Gazebo/robots/infantry.urdf.xacro (robot description, xacro)
@@ -8,17 +8,27 @@
     name="base_link">
     <inertial>
-      <origin
-        xyz="-0.025782 0 0.025311"
-        rpy="0 0 0" />
-      <mass
-        value="25.625" />
-      <inertia
-        ixx="0.10311"
-        ixy="-9.0391E-05"
-        ixz="0.0071078"
-        iyy="0.24575"
-        iyz="2.1083E-05"
-        izz="0.32438" />
-    </inertial>
+    <origin
+    xyz="0 0 0"
+    rpy="0 0 0" />
+    <mass
+    value="25.625" />
+    <inertia
+    ixx="0.10311"
+    ixy="-9.0391E-05"
+    ixz="0.0071078"
+    iyy="0.24575"
+    iyz="2.1083E-05"
+    izz="0.32438" />
+    </inertial>
+    <collision>
+    <origin
+    xyz="0 0 0"
+    rpy="0 0 0" />
+    <geometry>
+    <box
+    size= "0.55 0.4 0.1"
+    />
+    </geometry>
+    </collision>
     <visual>
       <origin
@@ -35,15 +45,43 @@
       </material>
     </visual>
-    <collision>
-      <origin
-        xyz="0 0 0"
-        rpy="0 0 0" />
-      <geometry>
-        <box
-          size= "0.55 0.4 0.1"
-        />
-      </geometry>
-    </collision>
-  </link>
+  </link>
+  <!--<link-->
+          <!--name="base_footprint">-->
+    <!--<inertial>-->
+      <!--<origin-->
+              <!--xyz="-0.025782 0 0.025311"-->
+              <!--rpy="0 0 0" />-->
+      <!--<mass-->
+              <!--value="25.625" />-->
+      <!--<inertia-->
+              <!--ixx="0.10311"-->
+              <!--ixy="-9.0391E-05"-->
+              <!--ixz="0.0071078"-->
+              <!--iyy="0.24575"-->
+              <!--iyz="2.1083E-05"-->
+              <!--izz="0.32438" />-->
+    <!--</inertial>-->
+    <!--<collision>-->
+      <!--<origin-->
+              <!--xyz="0 0 0"-->
+              <!--rpy="0 0 0" />-->
+      <!--<geometry>-->
+        <!--<box-->
+                <!--size= "0.55 0.4 0.1"-->
+        <!--/>-->
+      <!--</geometry>-->
+    <!--</collision>-->
+  <!--</link>-->
+  <!--<joint-->
+          <!--name="base_link_to_base_foot_print"-->
+          <!--type="fixed">-->
+    <!--<origin-->
+            <!--xyz="0 0 0"-->
+            <!--rpy="0 0 0" />-->
+    <!--<parent-->
+            <!--link="base_link" />-->
+    <!--<child-->
+            <!--link="base_footprint" />-->
+  <!--</joint>-->
   <link
     name="br_wheel_link">
@@ -85,4 +123,12 @@
           length = "${wheel_width}" />
       </geometry>
+      <surface>
+        <friction>
+          <ode>
+            <mu>0.0</mu>
+            <mu2>0.0</mu2>
+          </ode>
+        </friction>
+      </surface>
     </collision>
   </link>
@@ -139,4 +185,12 @@
           length = "${wheel_width}" />
       </geometry>
+      <surface>
+        <friction>
+          <ode>
+            <mu>0.0</mu>
+            <mu2>0.0</mu2>
+          </ode>
+        </friction>
+      </surface>
     </collision>
   </link>
@@ -193,4 +247,12 @@
           length = "${wheel_width}" />
       </geometry>
+      <surface>
+        <friction>
+          <ode>
+            <mu>0.0</mu>
+            <mu2>0.0</mu2>
+          </ode>
+        </friction>
+      </surface>
     </collision>
   </link>
@@ -247,4 +309,12 @@
           length = "${wheel_width}" />
       </geometry>
+      <surface>
+        <friction>
+          <ode>
+            <mu>0.0</mu>
+            <mu2>0.0</mu2>
+          </ode>
+        </friction>
+      </surface>
     </collision>
   </link>
@@ -305,5 +375,5 @@
   <joint
     name="base_link_to_yaw_joint"
-    type="revolute">
+    type="fixed">
     <origin
       xyz="-0.017561 0 0.1342"
@@ -315,9 +385,9 @@
     <axis
       xyz="0 0 1" />
-    <limit
-      lower="-1.57"
-      upper="1.57"
-      effort="1000"
-      velocity="100" />
+    <!--<limit-->
+      <!--lower="-1.57"-->
+      <!--upper="1.57"-->
+      <!--effort="1000"-->
+      <!--velocity="100" />-->
   </joint>
   <link
@@ -374,6 +444,6 @@
       xyz="0 1 0" />
     <limit
-      lower="-0.35"
-      upper="0.35"
+      lower="-0.001"
+      upper="0.001"
       effort="1000"
       velocity="100" />

File: RoboRTS_Gazebo/robots/infantry.xacro (robot description, xacro)
@@ -3,4 +3,4 @@
         <xacro:include filename="$(find roborts_gazebo)/robots/infantry.urdf.xacro" />
         <xacro:include filename="$(find roborts_gazebo)/robots/infantry.gazebo.xacro" />
-        <xacro:include filename="$(find roborts_gazebo)/robots/infantry.transmission.xacro" />
+        <!--<xacro:include filename="$(find roborts_gazebo)/robots/infantry.transmission.xacro" />-->
 </robot>
