Commit message: 修改了地图,模型使之符合ICRA 2019

File: RoboRTS_Gazebo/robots/infantry.gazebo.xacro (robot description, xacro)
@@ -1,34 +1,37 @@
 <?xml version="1.0"?>
-<robot xmlns:xacro="http://www.ros.org/wiki/xacro"
-	name="infantry_xacro">
+<robot xmlns:xacro="http://www.ros.org/wiki/xacro" name="roborts_robot_xacro">
   <xacro:macro name="led_color" params="name">
-  <gazebo reference="fr_wheel_link">
-    <material>Gazebo/Black</material>
-    <turnGravityOff>false</turnGravityOff>
-  </gazebo>
-  <gazebo reference="fl_wheel_link">
-    <material>Gazebo/Black</material>
-    <turnGravityOff>false</turnGravityOff>
-  </gazebo>
-  <gazebo reference="br_wheel_link">
-    <material>Gazebo/Black</material>
-    <turnGravityOff>false</turnGravityOff>
-  </gazebo>
-  <gazebo reference="bl_wheel_link">
-    <material>Gazebo/Black</material>
-    <turnGravityOff>false</turnGravityOff>
-  </gazebo>
-  <gazebo reference="yaw_link">
-    <material>Gazebo/Black</material>
-    <turnGravityOff>false</turnGravityOff>
-  </gazebo>
-  <gazebo reference="pitch_link">
-    <material>Gazebo/Black</material>
-    <turnGravityOff>false</turnGravityOff>
-  </gazebo>
-  <!-- <gazebo reference="camera_link">
-    <material>Gazebo/Black</material>
-    <turnGravityOff>false</turnGravityOff>
-  </gazebo>  -->
+    <gazebo reference="fr_wheel_link">
+      <material>Gazebo/Black</material>
+      <turnGravityOff>false</turnGravityOff>
+    </gazebo>
+    <gazebo reference="fl_wheel_link">
+      <material>Gazebo/Black</material>
+      <turnGravityOff>false</turnGravityOff>
+    </gazebo>
+    <gazebo reference="br_wheel_link">
+      <material>Gazebo/Black</material>
+      <turnGravityOff>false</turnGravityOff>
+    </gazebo>
+    <gazebo reference="bl_wheel_link">
+      <material>Gazebo/Black</material>
+      <turnGravityOff>false</turnGravityOff>
+    </gazebo>
+    <gazebo reference="yaw_link">
+      <material>Gazebo/Black</material>
+      <turnGravityOff>false</turnGravityOff>
+    </gazebo>
+    <gazebo reference="pitch_link">
+      <material>Gazebo/Black</material>
+      <turnGravityOff>false</turnGravityOff>
+    </gazebo>
+    <gazebo reference="camera_link">
+      <material>Gazebo/Black</material>
+      <turnGravityOff>false</turnGravityOff>
+    </gazebo>
+    <gazebo reference="led_link">
+      <material>Gazebo/${name}</material>
+      <turnGravityOff>false</turnGravityOff>
+    </gazebo>
   </xacro:macro>
   <!-- materials -->
@@ -82,4 +85,44 @@
     </sensor>
   </gazebo>
+  <!-- camera -->
+  <gazebo reference="camera_link">
+    <sensor type="camera" name="camera">
+      <update_rate>30.0</update_rate>
+      <camera name="head">
+        <horizontal_fov>1.3962634</horizontal_fov>
+        <image>
+          <width>640</width>
+          <height>480</height>
+          <format>R8G8B8</format>
+        </image>
+        <clip>
+          <near>0.02</near>
+          <far>300</far>
+        </clip>
+        <noise>
+          <type>gaussian</type>
+          <!-- Noise is sampled independently per pixel on each frame.
+               That pixel's noise value is added to each of its color
+               channels, which at that point lie in the range [0,1]. -->
+          <mean>0.0</mean>
+          <stddev>0.007</stddev>
+        </noise>
+      </camera>
+      <plugin name="camera_controller" filename="libgazebo_ros_camera.so">
+        <alwaysOn>true</alwaysOn>
+        <updateRate>0.0</updateRate>
+        <cameraName>robot/camera</cameraName>
+        <imageTopicName>image_raw</imageTopicName>
+        <cameraInfoTopicName>camera_info</cameraInfoTopicName>
+        <frameName>camera_Link</frameName>
+        <hackBaseline>0.07</hackBaseline>
+        <distortionK1>0.0</distortionK1>
+        <distortionK2>0.0</distortionK2>
+        <distortionK3>0.0</distortionK3>
+        <distortionT1>0.0</distortionT1>
+        <distortionT2>0.0</distortionT2>
+      </plugin>
+    </sensor>
+  </gazebo>
   <!-- position controller plugin-->
   <gazebo>
@@ -92,19 +135,6 @@
       <publish_odom_tf>1</publish_odom_tf>
       <rotation_velocity_p_gain>800.0</rotation_velocity_p_gain>
-   </plugin>
- </gazebo>
-  <!--<gazebo>-->
-  <!--<plugin name="mecanum_base_controller" filename="libroborts_gazebo_ros_force_based_move.so">-->
-  <!--<commandTopic>/cmd_vel</commandTopic>-->
-  <!--<odometryTopic>odom</odometryTopic>-->
-  <!--<odometryFrame>odom</odometryFrame>-->
-  <!--<odometryRate>20.0</odometryRate>-->
-  <!--<robotBaseFrame>base_link</robotBaseFrame>-->
-  <!--<yaw_velocity_p_gain>500</yaw_velocity_p_gain>-->
-  <!--<x_velocity_p_gain>3000</x_velocity_p_gain>-->
-  <!--<y_velocity_p_gain>3000</y_velocity_p_gain>-->
-  <!--<publishOdometryTf>1</publishOdometryTf>-->
-  <!--</plugin>-->
-  <!--</gazebo>-->
+    </plugin>
+  </gazebo>
   <gazebo>
     <plugin name="uwb_plugin" filename="libroborts_gazebo_ros_uwb.so">
@@ -135,10 +165,10 @@
     </sensor>
   </gazebo>
-<!-- ros_control plugin -->
-  <!--<gazebo>-->
-    <!--<plugin name="gazebo_ros_control" filename="libgazebo_ros_control.so">-->
-      <!--<robotParam>robot_description</robotParam>-->
-     <!-- <robotSimType>gazebo_ros_control/DefaultRobotHWSim</robotSimType>-->
-    <!--</plugin>-->
-  <!--</gazebo>-->
+  <!-- ros_control plugin -->
+  <gazebo>
+    <plugin name="gazebo_ros_control" filename="libgazebo_ros_control.so">
+      <robotParam>robot_description</robotParam>
+      <robotSimType>gazebo_ros_control/DefaultRobotHWSim</robotSimType>
+    </plugin>
+  </gazebo>
 </robot>

File: RoboRTS_Gazebo/robots/infantry.transmission.xacro (robot description, xacro)
@@ -1,23 +1,24 @@
 <?xml version="1.0"?>
-<robot name="infantry_xacro" xmlns:xacro="http://www.ros.org/wiki/xacro">
-<!-- Macro Transmissions for ROS Control -->
-    <xacro:macro name="transmission_block" params="joint_name">
-	  <transmission name="${joint_name}_tran1">
-	    <type>transmission_interface/SimpleTransmission</type>
-	    <joint name="${joint_name}">
-	      <hardwareInterface>hardware_interface/PositionJointInterface</hardwareInterface>
-            </joint>
-	    <actuator name="${joint_name}_motor1">
-              <mechanicalReduction>1</mechanicalReduction>
-	      <hardwareInterface>hardware_interface/PositionJointInterface</hardwareInterface>
-	    </actuator>
-	  </transmission>
-   </xacro:macro>
-<!-- Transmissions for ROS Control -->
-   <xacro:transmission_block joint_name="base_link_to_yaw_joint"/>
-   <xacro:transmission_block joint_name="base_link_to_pitch_joint"/>
-   <xacro:transmission_block joint_name="base_link_to_fl_wheel_joint"/>
-   <xacro:transmission_block joint_name="base_link_to_fr_wheel_joint"/>
-   <xacro:transmission_block joint_name="base_link_to_bl_wheel_joint"/>
-   <xacro:transmission_block joint_name="base_link_to_br_wheel_joint"/>
+<robot name="roborts_robot_xacro"
+  xmlns:xacro="http://www.ros.org/wiki/xacro">
+  <!-- Macro Transmissions for ROS Control -->
+  <xacro:macro name="transmission_block" params="joint_name">
+    <transmission name="${joint_name}_tran1">
+      <type>transmission_interface/SimpleTransmission</type>
+      <joint name="${joint_name}">
+        <hardwareInterface>hardware_interface/PositionJointInterface</hardwareInterface>
+      </joint>
+      <actuator name="${joint_name}_motor1">
+        <mechanicalReduction>1</mechanicalReduction>
+        <hardwareInterface>hardware_interface/PositionJointInterface</hardwareInterface>
+      </actuator>
+    </transmission>
+  </xacro:macro>
+  <!-- Transmissions for ROS Control -->
+  <xacro:transmission_block joint_name="base_link_to_yaw_joint"/>
+  <xacro:transmission_block joint_name="base_link_to_pitch_joint"/>
+  <xacro:transmission_block joint_name="base_link_to_fl_wheel_joint"/>
+  <xacro:transmission_block joint_name="base_link_to_fr_wheel_joint"/>
+  <xacro:transmission_block joint_name="base_link_to_bl_wheel_joint"/>
+  <xacro:transmission_block joint_name="base_link_to_br_wheel_joint"/>
 </robot>

File: RoboRTS_Gazebo/robots/infantry.urdf.xacro (robot description, xacro)
@@ -1,121 +1,43 @@
 <?xml version="1.0"?>
-<robot xmlns:xacro="http://www.ros.org/wiki/xacro" 	name="infantry_xacro">
-<xacro:property name="wheel_axe_width" value="0.25" />
-<xacro:property name="wheel_axe_length" value="0.21" />
-<xacro:property name="wheel_radius" value="0.078" />
-<xacro:property name="wheel_width" value="0.02" />
-  <link
-    name="base_link">
-    <inertial>
-    <origin
-    xyz="0 0 0"
-    rpy="0 0 0" />
-    <mass
-    value="25.625" />
-    <inertia
-    ixx="0.10311"
-    ixy="-9.0391E-05"
-    ixz="0.0071078"
-    iyy="0.24575"
-    iyz="2.1083E-05"
-    izz="0.32438" />
-    </inertial>
-    <collision>
-    <origin
-    xyz="0 0 0"
-    rpy="0 0 0" />
-    <geometry>
-    <box
-    size= "0.55 0.4 0.1"
-    />
-    </geometry>
-    </collision>
-    <visual>
-      <origin
-        xyz="0 0 0"
-        rpy="0 0 0" />
-      <geometry>
-        <mesh
-          filename="package://roborts_gazebo/meshes/base_link.STL" />
-      </geometry>
-      <material
-        name="">
-        <color
-          rgba="0 0 0 1" />
-      </material>
-    </visual>
-  </link>
-  <!--<link-->
-          <!--name="base_footprint">-->
-    <!--<inertial>-->
-      <!--<origin-->
-              <!--xyz="-0.025782 0 0.025311"-->
-              <!--rpy="0 0 0" />-->
-      <!--<mass-->
-              <!--value="25.625" />-->
-      <!--<inertia-->
-              <!--ixx="0.10311"-->
-              <!--ixy="-9.0391E-05"-->
-              <!--ixz="0.0071078"-->
-              <!--iyy="0.24575"-->
-              <!--iyz="2.1083E-05"-->
-              <!--izz="0.32438" />-->
-    <!--</inertial>-->
-    <!--<collision>-->
-      <!--<origin-->
-              <!--xyz="0 0 0"-->
-              <!--rpy="0 0 0" />-->
-      <!--<geometry>-->
-        <!--<box-->
-                <!--size= "0.55 0.4 0.1"-->
-        <!--/>-->
-      <!--</geometry>-->
-    <!--</collision>-->
-  <!--</link>-->
-  <!--<joint-->
-          <!--name="base_link_to_base_foot_print"-->
-          <!--type="fixed">-->
-    <!--<origin-->
-            <!--xyz="0 0 0"-->
-            <!--rpy="0 0 0" />-->
-    <!--<parent-->
-            <!--link="base_link" />-->
-    <!--<child-->
-            <!--link="base_footprint" />-->
-  <!--</joint>-->
-  <link
-    name="br_wheel_link">
-    <inertial>
-      <origin
-        xyz="0 0.014616 0"
-        rpy="0 0 0" />
-      <mass
-        value="0.86078" />
-      <inertia
-        ixx="0.0015361"
-        ixy="1.6456E-06"
-        ixz="-2.0131E-06"
-        iyy="0.002844"
-        iyz="-9.5351E-07"
-        izz="0.0015337" />
-    </inertial>
-    <visual>
-      <origin
-        xyz="0 0 0"
-        rpy="0 0 0" />
-      <geometry>
-        <mesh
-          filename="package://roborts_gazebo/meshes/br_wheel_link.STL" />
-      </geometry>
-      <material
-        name="">
-        <color
-          rgba="1 0 0 1" />
-      </material>
-    </visual>
-    <collision>
-      <origin
-        xyz="0 0 0"
-        rpy="1.5708 0 0" />
+<robot xmlns:xacro="http://www.ros.org/wiki/xacro" name="roborts_robot_xacro">
+  <xacro:property name="wheel_axe_width" value="0.25" />
+  <xacro:property name="wheel_axe_length" value="0.21" />
+  <xacro:property name="wheel_radius" value="0.078" />
+  <xacro:property name="wheel_width" value="0.02" />
+  <link name="base_link">
+    <inertial>
+      <origin xyz="0 0 0" rpy="0 0 0" />
+      <mass value="25.625" />
+      <inertia ixx="0.10311" ixy="-9.0391E-05" ixz="0.0071078" iyy="0.24575" iyz="2.1083E-05" izz="0.32438" />
+    </inertial>
+    <collision>
+      <origin xyz="0 0 0" rpy="0 0 0" />
+      <geometry>
+        <box size= "0.55 0.4 0.1" />
+      </geometry>
+    </collision>
+    <visual>
+      <origin xyz="0 0 0" rpy="0 0 0" />
+      <geometry>
+        <mesh filename="package://roborts_gazebo/meshes/base_link.STL" />
+      </geometry>
+      <material name="black"/>
+    </visual>
+  </link>
+  <link name="br_wheel_link">
+    <inertial>
+      <origin xyz="0 0.014616 0" rpy="0 0 0" />
+      <mass value="0.86078" />
+      <inertia ixx="0.0015361" ixy="1.6456E-06" ixz="-2.0131E-06" iyy="0.002844" iyz="-9.5351E-07" izz="0.0015337" />
+    </inertial>
+    <visual>
+      <origin xyz="0 0 0" rpy="0 0 0" />
+      <geometry>
+        <mesh filename="package://roborts_gazebo/meshes/br_wheel_link.STL" />
+      </geometry>
+      <material name="black"/>
+    </visual>
+    <collision>
+      <origin xyz="0 0 0" rpy="1.5708 0 0" />
       <geometry>
         <cylinder
@@ -133,51 +55,25 @@
     </collision>
   </link>
-  <joint
-    name="base_link_to_br_wheel_joint"
-    type="continuous">
-    <origin
-      xyz="-${wheel_axe_length} -${wheel_axe_width} 0"
-      rpy="0 0 -3.1416" />
-    <parent
-      link="base_link" />
-    <child
-      link="br_wheel_link" />
-    <axis
-      xyz="0 1 0" />
-  </joint>
-  <link
-    name="bl_wheel_link">
-    <inertial>
-      <origin
-        xyz="0 -0.014551 0"
-        rpy="0 0 0" />
-      <mass
-        value="0.86078" />
-      <inertia
-        ixx="0.0015355"
-        ixy="4.8831E-07"
-        ixz="1.8067E-06"
-        iyy="0.002844"
-        iyz="9.4618E-08"
-        izz="0.0015338" />
-    </inertial>
-    <visual>
-      <origin
-        xyz="0 0 0"
-        rpy="0 0 0" />
-      <geometry>
-        <mesh
-          filename="package://roborts_gazebo/meshes/bl_wheel_link.STL" />
-      </geometry>
-      <material
-        name="">
-        <color
-          rgba="0.79216 0.81961 0.93333 1" />
-      </material>
-    </visual>
-    <collision>
-      <origin
-        xyz="0 0 0"
-        rpy="-1.5708 0 0" />
+  <joint name="base_link_to_br_wheel_joint" type="continuous">
+    <origin xyz="-${wheel_axe_length} -${wheel_axe_width} 0" rpy="0 0 -3.1416" />
+    <parent link="base_link" />
+    <child link="br_wheel_link" />
+    <axis xyz="0 1 0" />
+  </joint>
+  <link name="bl_wheel_link">
+    <inertial>
+      <origin xyz="0 -0.014551 0" rpy="0 0 0" />
+      <mass value="0.86078" />
+      <inertia ixx="0.0015355" ixy="4.8831E-07" ixz="1.8067E-06" iyy="0.002844" iyz="9.4618E-08" izz="0.0015338" />
+    </inertial>
+    <visual>
+      <origin xyz="0 0 0" rpy="0 0 0" />
+      <geometry>
+        <mesh filename="package://roborts_gazebo/meshes/bl_wheel_link.STL" />
+      </geometry>
+      <material name="black"/>
+    </visual>
+    <collision>
+      <origin xyz="0 0 0" rpy="-1.5708 0 0" />
       <geometry>
         <cylinder
@@ -195,51 +91,25 @@
     </collision>
   </link>
-  <joint
-    name="base_link_to_bl_wheel_joint"
-    type="continuous">
-    <origin
-      xyz="-${wheel_axe_length} ${wheel_axe_width} 0"
-      rpy="0 0 -3.1416" />
-    <parent
-      link="base_link" />
-    <child
-      link="bl_wheel_link" />
-    <axis
-      xyz="0 -1 0" />
-  </joint>
-  <link
-    name="fl_wheel_link">
-    <inertial>
-      <origin
-        xyz="0 -0.014549 0"
-        rpy="0 0 0" />
-      <mass
-        value="0.86078" />
-      <inertia
-        ixx="0.0015361"
-        ixy="1.6481E-06"
-        ixz="-2.0131E-06"
-        iyy="0.002844"
-        iyz="-9.4912E-07"
-        izz="0.0015338" />
-    </inertial>
-    <visual>
-      <origin
-        xyz="0 0 0"
-        rpy="0 0 0" />
-      <geometry>
-        <mesh
-          filename="package://roborts_gazebo/meshes/fl_wheel_link.STL" />
-      </geometry>
-      <material
-        name="">
-        <color
-          rgba="0.79216 0.81961 0.93333 1" />
-      </material>
-    </visual>
-    <collision>
-       <origin
-        xyz="0 0 0"
-        rpy="-1.5708 0 0" />
+  <joint name="base_link_to_bl_wheel_joint" type="continuous">
+    <origin xyz="-${wheel_axe_length} ${wheel_axe_width} 0" rpy="0 0 -3.1416" />
+    <parent link="base_link" />
+    <child link="bl_wheel_link" />
+    <axis xyz="0 -1 0" />
+  </joint>
+  <link name="fl_wheel_link">
+    <inertial>
+      <origin xyz="0 -0.014549 0" rpy="0 0 0" />
+      <mass value="0.86078" />
+      <inertia ixx="0.0015361" ixy="1.6481E-06" ixz="-2.0131E-06" iyy="0.002844" iyz="-9.4912E-07" izz="0.0015338" />
+    </inertial>
+    <visual>
+      <origin xyz="0 0 0" rpy="0 0 0" />
+      <geometry>
+        <mesh filename="package://roborts_gazebo/meshes/fl_wheel_link.STL" />
+      </geometry>
+      <material name="black"/>
+    </visual>
+    <collision>
+      <origin xyz="0 0 0" rpy="-1.5708 0 0" />
       <geometry>
         <cylinder
@@ -257,51 +127,25 @@
     </collision>
   </link>
-  <joint
-    name="base_link_to_fl_wheel_joint"
-    type="continuous">
-    <origin
-      xyz="${wheel_axe_length} ${wheel_axe_width} 0"
-      rpy="0 0 3.1416" />
-    <parent
-      link="base_link" />
-    <child
-      link="fl_wheel_link" />
-    <axis
-      xyz="0 1 0" />
-  </joint>
-  <link
-    name="fr_wheel_link">
-    <inertial>
-      <origin
-        xyz="0.00010086 0.014592 0"
-        rpy="0 0 0" />
-      <mass
-        value="0.86078" />
-      <inertia
-        ixx="0.0015355"
-        ixy="5.3543E-07"
-        ixz="1.8067E-06"
-        iyy="0.002844"
-        iyz="1.1717E-07"
-        izz="0.0015337" />
-    </inertial>
-    <visual>
-      <origin
-        xyz="0 0 0"
-        rpy="0 0 0" />
-      <geometry>
-        <mesh
-          filename="package://roborts_gazebo/meshes/fr_wheel_link.STL" />
-      </geometry>
-      <material
-        name="">
-        <color
-          rgba="0.75294 0.75294 0.75294 1" />
-      </material>
-    </visual>
-    <collision>
-      <origin
-        xyz="0 0 0"
-        rpy="1.5708 0 0" />
+  <joint name="base_link_to_fl_wheel_joint" type="continuous">
+    <origin xyz="${wheel_axe_length} ${wheel_axe_width} 0" rpy="0 0 3.1416" />
+    <parent link="base_link" />
+    <child link="fl_wheel_link" />
+    <axis xyz="0 1 0" />
+  </joint>
+  <link name="fr_wheel_link">
+    <inertial>
+      <origin xyz="0.00010086 0.014592 0" rpy="0 0 0" />
+      <mass value="0.86078" />
+      <inertia ixx="0.0015355" ixy="5.3543E-07" ixz="1.8067E-06" iyy="0.002844" iyz="1.1717E-07" izz="0.0015337" />
+    </inertial>
+    <visual>
+      <origin xyz="0 0 0" rpy="0 0 0" />
+      <geometry>
+        <mesh filename="package://roborts_gazebo/meshes/fr_wheel_link.STL" />
+      </geometry>
+      <material name="black"/>
+    </visual>
+    <collision>
+      <origin xyz="0 0 0" rpy="1.5708 0 0" />
       <geometry>
         <cylinder
@@ -319,339 +163,187 @@
     </collision>
   </link>
-  <joint
-    name="base_link_to_fr_wheel_joint"
-    type="continuous">
-    <origin
-      xyz="${wheel_axe_length} -${wheel_axe_width} 0"
-      rpy="0 0 -3.1416" />
-    <parent
-      link="base_link" />
-    <child
-      link="fr_wheel_link" />
-    <axis
-      xyz="0 -1 0" />
-  </joint>
-  <link
-    name="yaw_link">
-    <inertial>
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
File: RoboRTS_Gazebo/robots/infantry.xacro (robot description, xacro)
@@ -3,4 +3,5 @@
         <xacro:include filename="$(find roborts_gazebo)/robots/infantry.urdf.xacro" />
         <xacro:include filename="$(find roborts_gazebo)/robots/infantry.gazebo.xacro" />
-        <!--<xacro:include filename="$(find roborts_gazebo)/robots/infantry.transmission.xacro" />-->
+        <xacro:include filename="$(find roborts_gazebo)/robots/infantry.transmission.xacro" />
+        <xacro:led_color name="White"/>
 </robot>
